Commit message: update mecharm_pi urdf

File: mycobot_description/urdf/mecharm_pi/mecharm_pi.urdf (robot description, URDF)
Before this commit: robot firefighter, 7 links, 6 joints
Joints:
- joint joint2_to_joint1: limit lower=-1.570796 upper=1.570796 effort=1000.0 velocity=0 -> lower=-1.48353 upper=1.570796 effort=1000.0 velocity=0; origin xyz=0 0 0.038 rpy= 1.5708 0 0  -> xyz=0 0 0.038 rpy= -1.5708 0 0 
- joint joint3_to_joint2: limit lower=-3.08 upper=0.785398 effort=1000.0 velocity=0 -> lower=-3.14 upper=0.785398 effort=1000.0 velocity=0; origin xyz=0.0 0.1 0    rpy=3.1415926 0 0  -> xyz=0.0 -0.1 0    rpy=0 0 0 
- joint joint5_to_joint4: origin xyz= -0.001 0 0.0 rpy=  0 -1.5708 3.1415926 -> xyz= -0.001 0 0.0 rpy=  0 -1.5708 0

Commit message: rename mecharm_pi to mecharm

File: mycobot_description/urdf/mecharm_pi/mecharm_pi.urdf (robot description, URDF)
Before this commit: robot firefighter, 7 links, 6 joints
Links:
- link base: geometry collision mesh filename=package://mycobot_description/urdf/mecharm/base.dae; visual mesh filename=package://mycobot_description/urdf/mecharm/base.dae
- link link1: geometry collision mesh filename=package://mycobot_description/urdf/mecharm/link1.dae; visual mesh filename=package://mycobot_description/urdf/mecharm/link1.dae
- link link2: geometry collision mesh filename=package://mycobot_description/urdf/mecharm/link2.dae; visual mesh filename=package://mycobot_description/urdf/mecharm/link2.dae
- link link3: geometry collision mesh filename=package://mycobot_description/urdf/mecharm/link3.dae; visual mesh filename=package://mycobot_description/urdf/mecharm/link3.dae
- link link4: geometry collision mesh filename=package://mycobot_description/urdf/mecharm/link4.dae; visual mesh filename=package://mycobot_description/urdf/mecharm/link4.dae
- link link5: geometry collision mesh filename=package://mycobot_description/urdf/mecharm/link5.dae; visual mesh filename=package://mycobot_description/urdf/mecharm/link5.dae
- link link6: geometry collision mesh filename=package://mycobot_description/urdf/mecharm/link6.dae; visual mesh filename=package://mycobot_description/urdf/mecharm/link6.dae
