Commit message: fix bug

File: mycobot_description/urdf/320_pi/mycobot_pro_320_pi.urdf (robot description, URDF)
Before this commit: robot firefighter, 7 links, 6 joints
Links:
- link base: geometry collision mesh filename=package://mycobot_description/urdf/320_pi/base.dae; visual mesh filename=package://mycobot_description/urdf/320_pi/base.dae
- link link1: geometry collision mesh filename=package://mycobot_description/urdf/320_pi/link1.dae; visual mesh filename=package://mycobot_description/urdf/320_pi/link1.dae
- link link2: geometry collision mesh filename=package://mycobot_description/urdf/320_pi/link2.dae; visual mesh filename=package://mycobot_description/urdf/320_pi/link2.dae
- link link3: geometry collision mesh filename=package://mycobot_description/urdf/320_pi/link3.dae; visual mesh filename=package://mycobot_description/urdf/320_pi/link3.dae
- link link4: geometry collision mesh filename=package://mycobot_description/urdf/320_pi/link4.dae; visual mesh filename=package://mycobot_description/urdf/320_pi/link4.dae
- link link5: geometry collision mesh filename=package://mycobot_description/urdf/320_pi/link5.dae; visual mesh filename=package://mycobot_description/urdf/320_pi/link5.dae
- link link6: geometry collision mesh filename=package://mycobot_description/urdf/320_pi/link6.dae; visual mesh filename=package://mycobot_description/urdf/320_pi/link6.dae
