Commit message: add mycobot_320_320 urdf

File: mycobot_description/urdf/320_urdf/mycobot_pro_320.urdf (robot description, URDF)
Before this commit: robot firefighter, 8 links, 7 joints
Links:
- removed link gripper
- link base: geometry collision mesh filename=package://mycobot_description/urdf/320_urdf/base.dae; visual mesh filename=package://mycobot_description/urdf/320_urdf/base.dae
- link link1: geometry collision mesh filename=package://mycobot_description/urdf/320_urdf/link1.dae; visual mesh filename=package://mycobot_description/urdf/320_urdf/link1.dae
- link link2: geometry collision mesh filename=package://mycobot_description/urdf/320_urdf/link2.dae; visual mesh filename=package://mycobot_description/urdf/320_urdf/link2.dae
- link link3: geometry collision mesh filename=package://mycobot_description/urdf/320_urdf/link3.dae; visual mesh filename=package://mycobot_description/urdf/320_urdf/link3.dae
- link link4: geometry collision mesh filename=package://mycobot_description/urdf/320_urdf/link4.dae; visual mesh filename=package://mycobot_description/urdf/320_urdf/link4.dae
- link link5: geometry collision mesh filename=package://mycobot_description/urdf/320_urdf/link5.dae; visual mesh filename=package://mycobot_description/urdf/320_urdf/link5.dae
- link link6: geometry collision mesh filename=package://mycobot_description/urdf/320_urdf/link6.dae; visual mesh filename=package://mycobot_description/urdf/320_urdf/link6.dae
Joints:
- removed joint gitpper_to_joint6output
- joint joint2_to_joint1: limit lower=-3.14 upper=3.14159 effort=1000.0 velocity=0 -> lower=-2.96 upper=2.96 effort=1000.0 velocity=0; origin xyz=0 0 0.17846 rpy=0 0 0 -> xyz=0 0 0.162 rpy=0 0 0
- joint joint3_to_joint2: limit lower=-3.14 upper=3.14159 effort=1000.0 velocity=0 -> lower=-2.79 upper=2.79 effort=1000.0 velocity=0; origin xyz=0 0  0 rpy=0 -1.57080  1.57080 -> xyz=0 0 0 rpy=0 -1.5708 1.5708
- joint joint4_to_joint3: limit lower=-3.14 upper=3.14159 effort=1000.0 velocity=0 -> lower=-2.79 upper=2.79 effort=1000.0 velocity=0
- joint joint5_to_joint4: limit lower=-3.14 upper=3.14159 effort=1000.0 velocity=0 -> lower=-2.79 upper=2.79 effort=1000.0 velocity=0; origin xyz=0.1 0  0.090 rpy=0 0 1.57080 -> xyz=0.1205 0 0.082  rpy= 0 0 1.57080
- joint joint6_to_joint5: limit lower=-3.14 upper=3.14159 effort=1000.0 velocity=0 -> lower=-2.96 upper=2.96 effort=1000.0 velocity=0; origin xyz=0 -0.08515 0 rpy=1.57080 -1.57080 0 -> xyz=0 -0.084 0.0 rpy=1.5708 0 0
- joint joint6output_to_joint6: limit lower=-3.14 upper=3.14159 effort=1000.0 velocity=0 -> lower=-3.05 upper=3.05 effort=1000.0 velocity=0; origin xyz=0 0.06 0 rpy=-1.57080 0 0  -> xyz=0 0.06635 0.0 rpy=-1.5708 0 0

Commit message: update 2022 version 320 ROS2 urdf model file

File: mycobot_description/urdf/320_urdf/mycobot_pro_320.urdf (robot description, URDF)
Before this commit: robot firefighter, 7 links, 6 joints
Joints:
- joint joint2_to_joint1: limit lower=-2.96 upper=2.96 effort=1000.0 velocity=0 -> lower=-2.87 upper=2.87 effort=1000.0 velocity=0; origin xyz=0 0 0.162 rpy=0 0 0 -> xyz=0 0 0.173 rpy=0 0 0
- joint joint3_to_joint2: limit lower=-2.79 upper=2.79 effort=1000.0 velocity=0 -> lower=-2.879 upper=2.879 effort=1000.0 velocity=0; origin xyz=0 0 0 rpy=0 -1.5708 1.5708 -> xyz=0 -0.086 0 rpy=0 -1.5708 1.5708
- joint joint4_to_joint3: limit lower=-2.79 upper=2.79 effort=1000.0 velocity=0 -> lower=-2.879 upper=2.879 effort=1000.0 velocity=0; origin xyz=0.13635 0 0    rpy=0 0 0 -> xyz=0.13635 0 -0.086    rpy=0 0 0
- joint joint5_to_joint4: limit lower=-2.79 upper=2.79 effort=1000.0 velocity=0 -> lower=-2.879 upper=2.879 effort=1000.0 velocity=0; origin xyz=0.1205 0 0.082  rpy= 0 0 1.57080 -> xyz=0.1195 0 0.082  rpy= 0 0 1.57080
- joint joint6_to_joint5: limit lower=-2.96 upper=2.96 effort=1000.0 velocity=0 -> lower=-2.879 upper=2.879 effort=1000.0 velocity=0; origin xyz=0 -0.084 0.0 rpy=1.5708 0 0 -> xyz=0 -0.09415 0.0 rpy=1.5708 0 0
- joint joint6output_to_joint6: origin xyz=0 0.06635 0.0 rpy=-1.5708 0 0 -> xyz=0 0.055 0.0 rpy=-1.5708 0 0
