Commit message: fix cobotx a450 urdf model for joint7

File: mycobot_description/urdf/cobotx_a450/cobotx_a450.urdf (robot description, URDF)
Before this commit: robot firefighter, 8 links, 7 joints
Joints:
- joint joint7_to_joint6: origin xyz=0.038 -0.046 0 rpy=-1.5708 0 0 -> xyz=0.038 -0.046 0 rpy=1.5708 0 0
