Commit message: 增加280M5、280PI ros 摄像头模组配置和吸泵配置

File: mycobot_description/urdf/mycobot/mycobot_urdf.urdf (robot description, URDF)
Before this commit: robot firefighter, 7 links, 6 joints
Links:
- added link g_base; collision mesh filename=package://mycobot_description/urdf/mycobot/G_base.dae; visual mesh filename=package://mycobot_description/urdf/mycobot/G_base.dae
Joints:
- added joint g_base_to_joint1: type fixed, parent g_base, child joint1, origin xyz=0 0 0 rpy=0 0 0, axis 0 0 0, limit lower=-3.14 upper=3.14159 effort=1000.0 velocity=0

File: mycobot_description/urdf/mycobot_pi/mycobot_urdf.urdf (robot description, URDF)
Before this commit: robot firefighter, 7 links, 6 joints
Links:
- added link g_base; collision mesh filename=package://mycobot_description/urdf/mycobot_pi/G_base.dae; visual mesh filename=package://mycobot_description/urdf/mycobot_pi/G_base.dae
Joints:
- added joint g_base_to_joint1: type fixed, parent g_base, child joint1, origin xyz=0 0 0 rpy=0 0 0, axis 0 0 0, limit lower=-3.14 upper=3.14159 effort=1000.0 velocity=0
