Commit message: 将 ros中cobotx相关的名称重命名为mercury

File: mycobot_description/urdf/mercury_a1/mercury_a1.urdf (robot description, URDF)
Before this commit: robot firefighter, 8 links, 7 joints
Links:
- link base: geometry collision mesh filename=package://mycobot_description/urdf/mercury_a1/base.dae; visual mesh filename=package://mycobot_description/urdf/mercury_a1/base.dae
- link joint1: geometry collision mesh filename=package://mycobot_description/urdf/mercury_a1/joint1.dae; visual mesh filename=package://mycobot_description/urdf/mercury_a1/joint1.dae
- link joint2: geometry collision mesh filename=package://mycobot_description/urdf/mercury_a1/joint2.dae; visual mesh filename=package://mycobot_description/urdf/mercury_a1/joint2.dae
- link joint3: geometry collision mesh filename=package://mycobot_description/urdf/mercury_a1/joint3.dae; visual mesh filename=package://mycobot_description/urdf/mercury_a1/joint3.dae
- link joint4: geometry collision mesh filename=package://mycobot_description/urdf/mercury_a1/joint4.dae; visual mesh filename=package://mycobot_description/urdf/mercury_a1/joint4.dae
- link joint5: geometry collision mesh filename=package://mycobot_description/urdf/mercury_a1/joint5.dae; visual mesh filename=package://mycobot_description/urdf/mercury_a1/joint5.dae
- link joint6: geometry collision mesh filename=package://mycobot_description/urdf/mercury_a1/joint6.dae; visual mesh filename=package://mycobot_description/urdf/mercury_a1/joint6.dae
- link joint7: geometry collision mesh filename=package://mycobot_description/urdf/mercury_a1/joint7.dae; visual mesh filename=package://mycobot_description/urdf/mercury_a1/joint7.dae
