Commit message: add pro 600 ROS2 use

File: mycobot_description/urdf/600_urdf/mycobot_600_urdf.urdf (robot description, URDF)
Before this commit: robot firefighter, 7 links, 6 joints
Joints:
- joint joint3_to_joint2: limit lower=-3.14 upper=3.14159 effort=1000.0 velocity=0 -> lower=-4.7123 upper=1.5708 effort=1000.0 velocity=0
- joint joint4_to_joint3: limit lower=-3.14 upper=3.14159 effort=1000.0 velocity=0 -> lower=-2.6179 upper=2.443 effort=1000.0 velocity=0
- joint joint5_to_joint4: limit lower=-3.14 upper=3.14159 effort=1000.0 velocity=0 -> lower=-4.5378 upper=1.3962 effort=1000.0 velocity=0
- joint joint6_to_joint5: limit lower=-3.14 upper=3.14159 effort=1000.0 velocity=0 -> lower=-2.9321 upper=2.9321 effort=1000.0 velocity=0
- joint joint6output_to_joint6: limit lower=-3.14 upper=3.14159 effort=1000.0 velocity=0 -> lower=-3.0368 upper=3.0368 effort=1000.0 velocity=0
