Commit message: update mycobot 630 urdf

File: mycobot_description/urdf/mycobot_630/mycobot_630.urdf (robot description, URDF)
Before this commit: robot firefighter, 7 links, 6 joints
Links:
- link base: geometry collision mesh filename=package://mycobot_description/urdf/mycobot_630/base.dae; visual mesh filename=package://mycobot_description/urdf/mycobot_630/base.dae
- link link1: geometry collision mesh filename=package://mycobot_description/urdf/mycobot_630/link1.dae; visual mesh filename=package://mycobot_description/urdf/mycobot_630/link1.dae
- link link2: geometry collision mesh filename=package://mycobot_description/urdf/mycobot_630/link2.dae; visual mesh filename=package://mycobot_description/urdf/mycobot_630/link2.dae
- link link3: geometry collision mesh filename=package://mycobot_description/urdf/mycobot_630/link3.dae; visual mesh filename=package://mycobot_description/urdf/mycobot_630/link3.dae
- link link4: geometry collision mesh filename=package://mycobot_description/urdf/mycobot_630/link4.dae; visual mesh filename=package://mycobot_description/urdf/mycobot_630/link4.dae
- link link5: geometry collision mesh filename=package://mycobot_description/urdf/mycobot_630/link5.dae; visual mesh filename=package://mycobot_description/urdf/mycobot_630/link5.dae
- link link6: geometry collision mesh filename=package://mycobot_description/urdf/mycobot_630/link6.dae; visual mesh filename=package://mycobot_description/urdf/mycobot_630/link6.dae
Joints:
- removed joint joint6output_to_joint6
- added joint joint1_to_base: type revolute, parent base, child link1, origin xyz=0 0 0.22934 rpy=0 0 0, axis 0 0 1, limit lower=-3.14 upper=3.14159 effort=1000.0 velocity=0
- joint joint2_to_joint1: axis 0 0 1 -> 0 0 -1; child link1 -> link2; limit lower=-3.14 upper=3.14159 effort=1000.0 velocity=0 -> lower=-4.71 upper=1.5707 effort=1000.0 velocity=0; origin xyz=0 0 0.19934 rpy=0 0 0 -> xyz=0 0  0 rpy=1.5707 0 0; parent base -> link1
- joint joint3_to_joint2: axis 0 0 -1 ->  0 0 -1; child link2 -> link3; limit lower=-4.7123 upper=1.5708 effort=1000.0 velocity=0 -> lower=-2.61 upper=2.618 effort=1000.0 velocity=0; origin xyz=0 0  0 rpy=1.5708 0 0 -> xyz=0.27 0 0    rpy=0 0 0; parent link1 -> link2
- joint joint4_to_joint3: child link3 -> link4; limit lower=-2.6179 upper=2.443 effort=1000.0 velocity=0 -> lower=-4.53 upper=1.3962 effort=1000.0 velocity=0; origin xyz=0.25 0 0    rpy=0 0 0 -> xyz=0.267 0  -0.0745 rpy=0 0 0; parent link2 -> link3
- joint joint5_to_joint4: axis  0 0 -1 -> 0 0 1; child link4 -> link5; limit lower=-4.5378 upper=1.3962 effort=1000.0 velocity=0 -> lower=-2.93 upper=2.9321 effort=1000.0 velocity=0; origin xyz=0.25 0  -0.1091 rpy=0 0 0 -> xyz=0 -0.095 0.002 rpy=1.5707 -1.5707 0; parent link3 -> link4
- joint joint6_to_joint5: axis 0 0 1 -> -1 0 0; child link5 -> link6; limit lower=-2.9321 upper=2.9321 effort=1000.0 velocity=0 -> lower=-3.03 upper=3.0368 effort=1000.0 velocity=0; origin xyz=0 -0.108 0 rpy=1.57080 -1.57080 0 -> xyz=-0.054 0 0 rpy=-1.5707 0 0 ; parent link4 -> link5
