Commit message: 更新适配x5pi代码，重命名为rdkx5

File: mycobot_description/urdf/mycobot_280_rdkx5/mycobot_280_rdkx5.urdf (robot description, URDF)
Before this commit: robot firefighter, 7 links, 6 joints
Links:
- link joint1: geometry collision mesh filename=package://mycobot_description/urdf/mycobot_280_rdkx5/joint1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; visual mesh filename=package://mycobot_description/urdf/mycobot_280_rdkx5/joint1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
- link joint2: geometry collision mesh filename=package://mycobot_description/urdf/mycobot_280_rdkx5/joint2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; visual mesh filename=package://mycobot_description/urdf/mycobot_280_rdkx5/joint2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
- link joint3: geometry collision mesh filename=package://mycobot_description/urdf/mycobot_280_rdkx5/joint3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; visual mesh filename=package://mycobot_description/urdf/mycobot_280_rdkx5/joint3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
- link joint4: geometry collision mesh filename=package://mycobot_description/urdf/mycobot_280_rdkx5/joint4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; visual mesh filename=package://mycobot_description/urdf/mycobot_280_rdkx5/joint4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
- link joint5: geometry collision mesh filename=package://mycobot_description/urdf/mycobot_280_rdkx5/joint5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; visual mesh filename=package://mycobot_description/urdf/mycobot_280_rdkx5/joint5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
- link joint6: geometry collision mesh filename=package://mycobot_description/urdf/mycobot_280_rdkx5/joint6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; visual mesh filename=package://mycobot_description/urdf/mycobot_280_rdkx5/joint6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
- link joint6_flange: geometry collision mesh filename=package://mycobot_description/urdf/mycobot_280_rdkx5/joint7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; visual mesh filename=package://mycobot_description/urdf/mycobot_280_rdkx5/joint7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
