Commit message: 重构musepi名字，改为risc-V

File: mycobot_description/urdf/mycobot_280_risc_v/mycobot_280_risc_v.urdf (robot description, URDF)
Before this commit: robot firefighter, 8 links, 7 joints
Links:
- link g_base: geometry collision mesh filename=package://mycobot_description/urdf/mycobot_280_risc_v/G_bas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; visual mesh filename=package://mycobot_description/urdf/mycobot_280_risc_v/G_bas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
- link joint1: geometry collision mesh filename=package://mycobot_description/urdf/mycobot_280_risc_v/joint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; visual mesh filename=package://mycobot_description/urdf/mycobot_280_risc_v/joint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
- link joint2: geometry collision mesh filename=package://mycobot_description/urdf/mycobot_280_risc_v/joint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; visual mesh filename=package://mycobot_description/urdf/mycobot_280_risc_v/joint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
- link joint3: geometry collision mesh filename=package://mycobot_description/urdf/mycobot_280_risc_v/joint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; visual mesh filename=package://mycobot_description/urdf/mycobot_280_risc_v/joint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
- link joint4: geometry collision mesh filename=package://mycobot_description/urdf/mycobot_280_risc_v/joint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; visual mesh filename=package://mycobot_description/urdf/mycobot_280_risc_v/joint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
- link joint5: geometry collision mesh filename=package://mycobot_description/urdf/mycobot_280_risc_v/joint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; visual mesh filename=package://mycobot_description/urdf/mycobot_280_risc_v/joint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
- link joint6: geometry collision mesh filename=package://mycobot_description/urdf/mycobot_280_risc_v/joint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; visual mesh filename=package://mycobot_description/urdf/mycobot_280_risc_v/joint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
- link joint6_flange: geometry collision mesh filename=package://mycobot_description/urdf/mycobot_280_risc_v/joint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; visual mesh filename=package://mycobot_description/urdf/mycobot_280_risc_v/joint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

File: mycobot_description/urdf/mycobot_280_risc_v/mycobot_280_risc_v_with_camera_flange.urdf (robot description, URDF)
Before this commit: robot firefighter, 9 links, 8 joints
Links:
- link camera_flange: geometry collision mesh filename=package://mycobot_description/urdf/mycobot_280_risc_v/camer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; visual mesh filename=package://mycobot_description/urdf/mycobot_280_risc_v/camer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
- link g_base: geometry collision mesh filename=package://mycobot_description/urdf/mycobot_280_risc_v/G_bas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; visual mesh filename=package://mycobot_description/urdf/mycobot_280_risc_v/G_bas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
- link joint1: geometry collision mesh filename=package://mycobot_description/urdf/mycobot_280_risc_v/joint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; visual mesh filename=package://mycobot_description/urdf/mycobot_280_risc_v/joint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
- link joint2: geometry collision mesh filename=package://mycobot_description/urdf/mycobot_280_risc_v/joint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; visual mesh filename=package://mycobot_description/urdf/mycobot_280_risc_v/joint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
- link joint3: geometry collision mesh filename=package://mycobot_description/urdf/mycobot_280_risc_v/joint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; visual mesh filename=package://mycobot_description/urdf/mycobot_280_risc_v/joint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
- link joint4: geometry collision mesh filename=package://mycobot_description/urdf/mycobot_280_risc_v/joint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; visual mesh filename=package://mycobot_description/urdf/mycobot_280_risc_v/joint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
- link joint5: geometry collision mesh filename=package://mycobot_description/urdf/mycobot_280_risc_v/joint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; visual mesh filename=package://mycobot_description/urdf/mycobot_280_risc_v/joint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
- link joint6: geometry collision mesh filename=package://mycobot_description/urdf/mycobot_280_risc_v/joint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; visual mesh filename=package://mycobot_description/urdf/mycobot_280_risc_v/joint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
- link joint6_flange: geometry collision mesh filename=package://mycobot_description/urdf/mycobot_280_risc_v/joint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; visual mesh filename=package://mycobot_description/urdf/mycobot_280_risc_v/joint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

File: mycobot_description/urdf/mycobot_280_risc_v/mycobot_280_risc_v_with_camera_flange_pump.urdf (robot description, URDF)
Before this commit: robot firefighter, 11 links, 10 joints
Links:
- link camera_flange: geometry collision mesh filename=package://mycobot_description/urdf/mycobot_280_risc_v/camer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; visual mesh filename=package://mycobot_description/urdf/mycobot_280_risc_v/camer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
- link g_base: geometry collision mesh filename=package://mycobot_description/urdf/mycobot_280_risc_v/G_bas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; visual mesh filename=package://mycobot_description/urdf/mycobot_280_risc_v/G_bas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
- link joint1: geometry collision mesh filename=package://mycobot_description/urdf/mycobot_280_risc_v/joint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; visual mesh filename=package://mycobot_description/urdf/mycobot_280_risc_v/joint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
- link joint2: geometry collision mesh filename=package://mycobot_description/urdf/mycobot_280_risc_v/joint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; visual mesh filename=package://mycobot_description/urdf/mycobot_280_risc_v/joint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
- link joint3: geometry collision mesh filename=package://mycobot_description/urdf/mycobot_280_risc_v/joint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; visual mesh filename=package://mycobot_description/urdf/mycobot_280_risc_v/joint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
- link joint4: geometry collision mesh filename=package://mycobot_description/urdf/mycobot_280_risc_v/joint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; visual mesh filename=package://mycobot_description/urdf/mycobot_280_risc_v/joint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
- link joint5: geometry collision mesh filename=package://mycobot_description/urdf/mycobot_280_risc_v/joint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; visual mesh filename=package://mycobot_description/urdf/mycobot_280_risc_v/joint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
- link joint6: geometry collision mesh filename=package://mycobot_description/urdf/mycobot_280_risc_v/joint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; visual mesh filename=package://mycobot_description/urdf/mycobot_280_risc_v/joint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
- link joint6_flange: geometry collision mesh filename=package://mycobot_description/urdf/mycobot_280_risc_v/joint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; visual mesh filename=package://mycobot_description/urdf/mycobot_280_risc_v/joint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
- link pump_box: geometry collision mesh filename=package://mycobot_description/urdf/mycobot_280_risc_v/pump_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; visual mesh filename=package://mycobot_description/urdf/mycobot_280_risc_v/pump_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
- link pump_head: geometry collision mesh filename=package://mycobot_description/urdf/mycobot_280_risc_v/pump_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; visual mesh filename=package://mycobot_description/urdf/mycobot_280_risc_v/pump_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

File: mycobot_description/urdf/mycobot_280_risc_v/mycobot_280_risc_v_with_pump.urdf (robot description, URDF)
Before this commit: robot firefighter, 10 links, 9 joints
Links:
- link g_base: geometry collision mesh filename=package://mycobot_description/urdf/mycobot_280_risc_v/G_bas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; visual mesh filename=package://mycobot_description/urdf/mycobot_280_risc_v/G_bas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
- link joint1: geometry collision mesh filename=package://mycobot_description/urdf/mycobot_280_risc_v/joint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; visual mesh filename=package://mycobot_description/urdf/mycobot_280_risc_v/joint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
- link joint2: geometry collision mesh filename=package://mycobot_description/urdf/mycobot_280_risc_v/joint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; visual mesh filename=package://mycobot_description/urdf/mycobot_280_risc_v/joint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
- link joint3: geometry collision mesh filename=package://mycobot_description/urdf/mycobot_280_risc_v/joint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; visual mesh filename=package://mycobot_description/urdf/mycobot_280_risc_v/joint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
- link joint4: geometry collision mesh filename=package://mycobot_description/urdf/mycobot_280_risc_v/joint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; visual mesh filename=package://mycobot_description/urdf/mycobot_280_risc_v/joint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
- link joint5: geometry collision mesh filename=package://mycobot_description/urdf/mycobot_280_risc_v/joint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; visual mesh filename=package://mycobot_description/urdf/mycobot_280_risc_v/joint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
- link joint6: geometry collision mesh filename=package://mycobot_description/urdf/mycobot_280_risc_v/joint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; visual mesh filename=package://mycobot_description/urdf/mycobot_280_risc_v/joint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
- link joint6_flange: geometry collision mesh filename=package://mycobot_description/urdf/mycobot_280_risc_v/joint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; visual mesh filename=package://mycobot_description/urdf/mycobot_280_risc_v/joint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
- link pump_box: geometry collision mesh filename=package://mycobot_description/urdf/mycobot_280_risc_v/pump_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; visual mesh filename=package://mycobot_description/urdf/mycobot_280_risc_v/pump_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
- link pump_head: geometry collision mesh filename=package://mycobot_description/urdf/mycobot_280_risc_v/pump_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; visual mesh filename=package://mycobot_description/urdf/mycobot_280_risc_v/pump_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
