Commit message: opt mycobot 320 RISCV ROS2

File: mycobot_description/urdf/mycobot_320_riscv/mycobot_320_riscv.urdf (robot description, URDF)
Before this commit: robot firefighter, 7 links, 6 joints
Links:
- link base: geometry collision mesh filename=package://mycobot_description/urdf/mycobot_320_riscv/base.d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; visual mesh filename=package://mycobot_description/urdf/mycobot_320_riscv/base.d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
- link link1: geometry collision mesh filename=package://mycobot_description/urdf/mycobot_320_riscv/link1.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; visual mesh filename=package://mycobot_description/urdf/mycobot_320_riscv/link1.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
- link link2: geometry collision mesh filename=package://mycobot_description/urdf/mycobot_320_riscv/link2.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; visual mesh filename=package://mycobot_description/urdf/mycobot_320_riscv/link2.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
- link link3: geometry collision mesh filename=package://mycobot_description/urdf/mycobot_320_riscv/link3.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; visual mesh filename=package://mycobot_description/urdf/mycobot_320_riscv/link3.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
- link link4: geometry collision mesh filename=package://mycobot_description/urdf/mycobot_320_riscv/link4.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; visual mesh filename=package://mycobot_description/urdf/mycobot_320_riscv/link4.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
- link link5: geometry collision mesh filename=package://mycobot_description/urdf/mycobot_320_riscv/link5.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; visual mesh filename=package://mycobot_description/urdf/mycobot_320_riscv/link5.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
- link link6: geometry collision mesh filename=package://mycobot_description/urdf/mycobot_320_riscv/link6.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; visual mesh filename=package://mycobot_description/urdf/mycobot_320_riscv/link6.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
