Commit message: opt mycobot 280 RISCV ROS2

File: mycobot_description/urdf/mycobot_280_riscv/mycobot_280_riscv.urdf (robot description, URDF)
Before this commit: robot firefighter, 8 links, 7 joints
Links:
- link g_base: geometry collision mesh filename=package://mycobot_description/urdf/mycobot_280_riscv/G_base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; visual mesh filename=package://mycobot_description/urdf/mycobot_280_riscv/G_base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
- link joint1: geometry collision mesh filename=package://mycobot_description/urdf/mycobot_280_riscv/joint1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; visual mesh filename=package://mycobot_description/urdf/mycobot_280_riscv/joint1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
- link joint2: geometry collision mesh filename=package://mycobot_description/urdf/mycobot_280_riscv/joint2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; visual mesh filename=package://mycobot_description/urdf/mycobot_280_riscv/joint2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
- link joint3: geometry collision mesh filename=package://mycobot_description/urdf/mycobot_280_riscv/joint3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; visual mesh filename=package://mycobot_description/urdf/mycobot_280_riscv/joint3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
- link joint4: geometry collision mesh filename=package://mycobot_description/urdf/mycobot_280_riscv/joint4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; visual mesh filename=package://mycobot_description/urdf/mycobot_280_riscv/joint4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
- link joint5: geometry collision mesh filename=package://mycobot_description/urdf/mycobot_280_riscv/joint5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; visual mesh filename=package://mycobot_description/urdf/mycobot_280_riscv/joint5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
- link joint6: geometry collision mesh filename=package://mycobot_description/urdf/mycobot_280_riscv/joint6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; visual mesh filename=package://mycobot_description/urdf/mycobot_280_riscv/joint6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
- link joint6_flange: geometry collision mesh filename=package://mycobot_description/urdf/mycobot_280_riscv/joint7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; visual mesh filename=package://mycobot_description/urdf/mycobot_280_riscv/joint7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

File: mycobot_description/urdf/mycobot_280_riscv/mycobot_280_riscv_with_camera_flange.urdf (robot description, URDF)
Before this commit: robot firefighter, 9 links, 8 joints
Links:
- link camera_flange: geometry collision mesh filename=package://mycobot_description/urdf/mycobot_280_riscv/camera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; visual mesh filename=package://mycobot_description/urdf/mycobot_280_riscv/camera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
- link g_base: geometry collision mesh filename=package://mycobot_description/urdf/mycobot_280_riscv/G_base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; visual mesh filename=package://mycobot_description/urdf/mycobot_280_riscv/G_base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
- link joint1: geometry collision mesh filename=package://mycobot_description/urdf/mycobot_280_riscv/joint1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; visual mesh filename=package://mycobot_description/urdf/mycobot_280_riscv/joint1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
- link joint2: geometry collision mesh filename=package://mycobot_description/urdf/mycobot_280_riscv/joint2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; visual mesh filename=package://mycobot_description/urdf/mycobot_280_riscv/joint2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
- link joint3: geometry collision mesh filename=package://mycobot_description/urdf/mycobot_280_riscv/joint3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; visual mesh filename=package://mycobot_description/urdf/mycobot_280_riscv/joint3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
- link joint4: geometry collision mesh filename=package://mycobot_description/urdf/mycobot_280_riscv/joint4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; visual mesh filename=package://mycobot_description/urdf/mycobot_280_riscv/joint4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
- link joint5: geometry collision mesh filename=package://mycobot_description/urdf/mycobot_280_riscv/joint5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; visual mesh filename=package://mycobot_description/urdf/mycobot_280_riscv/joint5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
- link joint6: geometry collision mesh filename=package://mycobot_description/urdf/mycobot_280_riscv/joint6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; visual mesh filename=package://mycobot_description/urdf/mycobot_280_riscv/joint6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
- link joint6_flange: geometry collision mesh filename=package://mycobot_description/urdf/mycobot_280_riscv/joint7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; visual mesh filename=package://mycobot_description/urdf/mycobot_280_riscv/joint7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

File: mycobot_description/urdf/mycobot_280_riscv/mycobot_280_riscv_with_camera_flange_pump.urdf (robot description, URDF)
Before this commit: robot firefighter, 10 links, 9 joints
Links:
- added link camera_flange; collision mesh filename=package://mycobot_description/urdf/mycobot_280_riscv/camera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; visual mesh filename=package://mycobot_description/urdf/mycobot_280_riscv/camera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
- link g_base: geometry collision mesh filename=package://mycobot_description/urdf/mycobot_280_riscv/G_base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; visual mesh filename=package://mycobot_description/urdf/mycobot_280_riscv/G_base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
- link joint1: geometry collision mesh filename=package://mycobot_description/urdf/mycobot_280_riscv/joint1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; visual mesh filename=package://mycobot_description/urdf/mycobot_280_riscv/joint1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
- link joint2: geometry collision mesh filename=package://mycobot_description/urdf/mycobot_280_riscv/joint2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; visual mesh filename=package://mycobot_description/urdf/mycobot_280_riscv/joint2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
- link joint3: geometry collision mesh filename=package://mycobot_description/urdf/mycobot_280_riscv/joint3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; visual mesh filename=package://mycobot_description/urdf/mycobot_280_riscv/joint3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
- link joint4: geometry collision mesh filename=package://mycobot_description/urdf/mycobot_280_riscv/joint4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; visual mesh filename=package://mycobot_description/urdf/mycobot_280_riscv/joint4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
- link joint5: geometry collision mesh filename=package://mycobot_description/urdf/mycobot_280_riscv/joint5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; visual mesh filename=package://mycobot_description/urdf/mycobot_280_riscv/joint5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
- link joint6: geometry collision mesh filename=package://mycobot_description/urdf/mycobot_280_riscv/joint6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; visual mesh filename=package://mycobot_description/urdf/mycobot_280_riscv/joint6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
- link joint6_flange: geometry collision mesh filename=package://mycobot_description/urdf/mycobot_280_riscv/joint7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; visual mesh filename=package://mycobot_description/urdf/mycobot_280_riscv/joint7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
- link pump_box: geometry collision mesh filename=package://mycobot_description/urdf/mycobot_280_riscv/pump_b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; visual mesh filename=package://mycobot_description/urdf/mycobot_280_riscv/pump_b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
- link pump_head: geometry collision mesh filename=package://mycobot_description/urdf/mycobot_280_riscv/pump_h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; visual mesh filename=package://mycobot_description/urdf/mycobot_280_riscv/pump_h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
Joints:
- added joint joint6output_to_camera_flange: type fixed, parent joint6_flange, child camera_flange, origin xyz=0 0 0.01 rpy=1.579 0 0
- joint joint6output_to_pump_head: origin xyz=0 0 0.01 rpy=1.579 0 0 -> xyz=0 0 0.01 rpy=-1.579 0 0; parent joint6_flange -> camera_flange

File: mycobot_description/urdf/mycobot_280_riscv/mycobot_280_riscv_with_pump.urdf (robot description, URDF)
Before this commit: robot firefighter, 11 links, 10 joints
Links:
- removed link camera_flange
- link g_base: geometry collision mesh filename=package://mycobot_description/urdf/mycobot_280_riscv/G_base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; visual mesh filename=package://mycobot_description/urdf/mycobot_280_riscv/G_base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
- link joint1: geometry collision mesh filename=package://mycobot_description/urdf/mycobot_280_riscv/joint1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; visual mesh filename=package://mycobot_description/urdf/mycobot_280_riscv/joint1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
- link joint2: geometry collision mesh filename=package://mycobot_description/urdf/mycobot_280_riscv/joint2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; visual mesh filename=package://mycobot_description/urdf/mycobot_280_riscv/joint2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
- link joint3: geometry collision mesh filename=package://mycobot_description/urdf/mycobot_280_riscv/joint3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; visual mesh filename=package://mycobot_description/urdf/mycobot_280_riscv/joint3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
- link joint4: geometry collision mesh filename=package://mycobot_description/urdf/mycobot_280_riscv/joint4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; visual mesh filename=package://mycobot_description/urdf/mycobot_280_riscv/joint4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
- link joint5: geometry collision mesh filename=package://mycobot_description/urdf/mycobot_280_riscv/joint5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; visual mesh filename=package://mycobot_description/urdf/mycobot_280_riscv/joint5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
- link joint6: geometry collision mesh filename=package://mycobot_description/urdf/mycobot_280_riscv/joint6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; visual mesh filename=package://mycobot_description/urdf/mycobot_280_riscv/joint6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
- link joint6_flange: geometry collision mesh filename=package://mycobot_description/urdf/mycobot_280_riscv/joint7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; visual mesh filename=package://mycobot_description/urdf/mycobot_280_riscv/joint7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
- link pump_box: geometry collision mesh filename=package://mycobot_description/urdf/mycobot_280_riscv/pump_b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; visual mesh filename=package://mycobot_description/urdf/mycobot_280_riscv/pump_b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
- link pump_head: geometry collision mesh filename=package://mycobot_description/urdf/mycobot_280_riscv/pump_h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; visual mesh filename=package://mycobot_description/urdf/mycobot_280_riscv/pump_h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
Joints:
- removed joint joint6output_to_camera_flange
- joint joint6output_to_pump_head: origin xyz=0 0 0.01 rpy=-1.579 0 0 -> xyz=0 0 0.01 rpy=1.579 0 0; parent camera_flange -> joint6_flange
