Commit message: feat(320M5 foxy):Added Pro adaptive gripper control program and corresponding URDF

File: mycobot_description/urdf/mycobot_320_m5_2022/mycobot_320_m5_2022.urdf (robot description, URDF)
Before this commit: robot firefighter, 7 links, 6 joints
Joints:
- joint joint2_to_joint1: limit lower=-2.9321 upper=2.9321 effort=1000.0 velocity=0 -> lower=-2.93 upper=2.93 effort=1000.0 velocity=0; origin xyz=0 0 0.173 rpy=0 0 0 -> xyz=0 0 0.1739 rpy=0 0 0
- joint joint3_to_joint2: limit lower=-2.3561 upper=2.3561 effort=1000.0 velocity=0 -> lower=-2.35 upper=2.35 effort=1000.0 velocity=0; origin xyz=0 -0.086 0 rpy=0 -1.5708 1.5708 -> xyz=0 -0.08878 0 rpy=0 -1.5708 1.5708
- joint joint4_to_joint3: limit lower=-2.5307 upper=2.5307 effort=1000.0 velocity=0 -> lower=-2.53 upper=2.53 effort=1000.0 velocity=0; origin xyz=0.13635 0 -0.086    rpy=0 0 0 -> xyz=0.135 0 -0.08878    rpy=0 0 0
- joint joint5_to_joint4: limit lower=-2.5830 upper=2.5830 effort=1000.0 velocity=0 -> lower=-2.53 upper=2.53 effort=1000.0 velocity=0; origin xyz=0.1195 0 0.082  rpy= 0 0 1.57080 -> xyz=0.120 0 0.08878  rpy= 0 0 1.57080
- joint joint6_to_joint5: limit lower=-2.9321 upper=2.9321 effort=1000.0 velocity=0 -> lower=-2.93 upper=2.93 effort=1000.0 velocity=0; origin xyz=0 -0.09415 0.0 rpy=1.5708 0 0 -> xyz=0 -0.095 0.0 rpy=1.5708 0 0
- joint joint6output_to_joint6: limit lower=-3.14159 upper=3.14159 effort=1000.0 velocity=0 -> lower=-3.14 upper=3.14 effort=1000.0 velocity=0; origin xyz=0 0.055 0.0 rpy=-1.5708 0 0 -> xyz=0 0.0655 0.0 rpy=-1.5708 0 0
