Commit message: fix(pro450-ros): fix GUI movement abnormality, add force-controlled gripper model to GUI control and keyboard control

File: mycobot_description/urdf/mycobot_pro_450/mycobot_pro_450.urdf (robot description, URDF)
Before this commit: robot firefighter, 7 links, 6 joints
Joints:
- joint joint3: origin xyz=-0.01 0 0.18   rpy=0 0 0 -> xyz=-0.01 0 0.18 rpy=0 0 0
- joint joint4: axis  1 0 0 -> 1 0 0

File: mycobot_description/urdf/mycobot_pro_450/mycobot_pro_450_force_gripper.urdf (robot description, URDF)
Before this commit: robot firefighter, 15 links, 14 joints
Joints:
- joint joint3: origin xyz=-0.01 0 0.18   rpy=0 0 0 -> xyz=-0.01 0 0.18 rpy=0 0 0

Commit message: feat(pro450-ros2): Updated DH parameters in URDF file, updated joint range of motion, and optimized model following function

File: mycobot_description/urdf/mycobot_pro_450/mycobot_pro_450.urdf (robot description, URDF)
Before this commit: robot firefighter, 7 links, 6 joints
Joints:
- joint joint1: limit lower=-2.8797 upper=2.8797 effort=1000.0 velocity=0 -> lower=-2.8274 upper=2.8274 effort=1000.0 velocity=0; origin xyz=-0.0045 0 0.155 rpy=0 0 0 -> xyz=0 0 0.210 rpy=0 0 0
- joint joint2: limit lower=-2.0943 upper=2.0943 effort=1000.0 velocity=0 -> lower=-2.1816 upper=2.1816 effort=1000.0 velocity=0; origin xyz=0.05 0 0.048 rpy=0 0 0 -> xyz=0 -0.048 0 rpy=0 0 -1.5708
- joint joint3: limit lower=-2.7576 upper=2.7576 effort=1000.0 velocity=0 -> lower=-2.6878 upper=2.6878 effort=1000.0 velocity=0; origin xyz=-0.01 0 0.18 rpy=0 0 0 -> xyz=-0.01 0 0.18   rpy=0 0 0
- joint joint4: axis 1 0 0 ->  1 0 0; limit lower=-2.8797 upper=2.8797 effort=1000.0 velocity=0 -> lower=-2.8274 upper=2.8274 effort=1000.0 velocity=0; origin xyz=0.0 0 0.1735 rpy=0 0 0 -> xyz=0 0 0.173 rpy=0 0 0
- joint joint5: limit lower=-2.8797 upper=2.8797 effort=1000.0 velocity=0 -> lower=-2.8274 upper=2.8274 effort=1000.0 velocity=0; origin xyz=0.046 0.0003 0.05 rpy=0 0 0 -> xyz=0.0455 0 0.097 rpy=0 0 0
- joint joint6: limit lower=-3.0543 upper=3.0543 effort=1000.0 velocity=0 -> lower=-2.8797 upper=2.8797 effort=1000.0 velocity=0; origin xyz=0 0.04 0.0435 rpy=0 0 1.5708 -> xyz=0 0.04 0 rpy=0 0 1.5708

File: mycobot_description/urdf/mycobot_pro_450/mycobot_pro_450_force_gripper.urdf (robot description, URDF)
Before this commit: robot firefighter, 15 links, 14 joints
Joints:
- joint joint1: limit lower=-2.8797 upper=2.8797 effort=1000.0 velocity=0 -> lower=-2.8274 upper=2.8274 effort=1000.0 velocity=0; origin xyz=-0.0045 0 0.155 rpy=0 0 0 -> xyz=0 0 0.210 rpy=0 0 0
- joint joint2: limit lower=-2.0943 upper=2.0943 effort=1000.0 velocity=0 -> lower=-2.1816 upper=2.1816 effort=1000.0 velocity=0; origin xyz=0.05 0 0.048 rpy=0 0 0 -> xyz=0.0 -0.048 0 rpy=0 0 -1.5708
- joint joint3: limit lower=-2.7576 upper=2.7576 effort=1000.0 velocity=0 -> lower=-2.6878 upper=2.6878 effort=1000.0 velocity=0; origin xyz=-0.01 0 0.18 rpy=0 0 0 -> xyz=-0.01 0 0.18   rpy=0 0 0
- joint joint4: limit lower=-2.8797 upper=2.8797 effort=1000.0 velocity=0 -> lower=-2.8274 upper=2.8274 effort=1000.0 velocity=0; origin xyz=0.0 0 0.1735 rpy=0 0 0 -> xyz=0 0 0.173 rpy=0 0 0
- joint joint5: limit lower=-2.8797 upper=2.8797 effort=1000.0 velocity=0 -> lower=-2.8274 upper=2.8274 effort=1000.0 velocity=0; origin xyz=0.046 0.0003 0.05 rpy=0 0 0 -> xyz=0.0455 0 0.097 rpy=0 0 0
- joint joint6: limit lower=-3.0543 upper=3.0543 effort=1000.0 velocity=0 -> lower=-2.8797 upper=2.8797 effort=1000.0 velocity=0; origin xyz=0 0.04 0.0435 rpy=0 0 1.5708 -> xyz=0 0.04 0 rpy=0 0 1.5708
