Commit message: fix(pro630-urdf):Repair DH parameters in 630 urdf file

File: mycobot_description/urdf/mycobot_pro_630/mycobot_pro_630.urdf (robot description, URDF)
Before this commit: robot firefighter, 7 links, 6 joints
Joints:
- joint joint1_to_base: origin xyz=0 0 0.22934 rpy=0 0 0 -> xyz=0 0 0.206 rpy=0 0 0
- joint joint2_to_joint1: origin xyz=0 0  0 rpy=1.5707 -1.5708 0 -> xyz=0 0 0 rpy=1.5707 -1.5708 0
- joint joint3_to_joint2: origin xyz=0.27 0 0    rpy=0 0 0 -> xyz=0.269 0.0 0  rpy=0 0 0
- joint joint4_to_joint3: origin xyz=0.267 0  -0.0745 rpy=0 0 1.5708 -> xyz=0.266 0  -0.0745 rpy=0 0 1.5708
- joint joint5_to_joint4: origin xyz=0 -0.095 0.002 rpy=1.5707 -1.5707 0 -> xyz=0 -0.1 0.002 rpy=1.5707 -1.5707 0
- joint joint6_to_joint5: origin xyz=-0.054 0 0 rpy=-1.5707 0 0  -> xyz=-0.054 0 -0.004 rpy=-3.14159 0 0 

Commit message: perf(630-urdf): Optimized 630 URDF file to adapt to the latest DH parameters.

File: mycobot_description/urdf/mycobot_pro_630/mycobot_pro_630.urdf (robot description, URDF)
Before this commit: robot firefighter, 7 links, 6 joints
Joints:
- joint joint1_to_base: origin xyz=0 0 0.206 rpy=0 0 0 -> xyz=0 0 0.205 rpy=0 0 0
- joint joint3_to_joint2: origin xyz=0.269 0.0 0  rpy=0 0 0 -> xyz=0.269 0 0  rpy=0 0 0
- joint joint4_to_joint3: origin xyz=0.266 0  -0.0745 rpy=0 0 1.5708 -> xyz=0.266 0  -0.088 rpy=0 0 1.5708
- joint joint5_to_joint4: origin xyz=0 -0.1 0.002 rpy=1.5707 -1.5707 0 -> xyz=0 -0.095 0 rpy=1.5707 -1.5707 0
- joint joint6_to_joint5: origin xyz=-0.054 0 -0.004 rpy=-3.14159 0 0  -> xyz=-0.053 0 0 rpy=-3.14159 0 3.14159 
