Commit message: fix(pro630-urdf):Fix the collision issue in MoveIt2 path planning and back up the URDF file without offset angle

File: mycobot_description/urdf/mycobot_pro_630/mycobot_pro_630_no_offset.urdf (robot description, URDF)
Before this commit: robot firefighter, 7 links, 6 joints
Joints:
- joint joint2_to_joint1: limit lower=-3.14159 upper=3.14159 effort=1000.0 velocity=0 -> lower=-4.71 upper=1.5707 effort=1000.0 velocity=0; origin xyz=0 0 0 rpy=1.5707 -1.5708 0 -> xyz=0 0 0 rpy=1.5707 0 0
- joint joint4_to_joint3: limit lower=-2.9670 upper=2.9670 effort=1000.0 velocity=0 -> lower=-4.53 upper=1.3962 effort=1000.0 velocity=0; origin xyz=0.266 0  -0.088 rpy=0 0 1.5708 -> xyz=0.266 0  -0.088 rpy=0 0 0
