Commit message: feat(p1-urdf): update urdf file

File: mycobot_description/urdf/ultraArm_p1/ultraArm_p1.urdf (robot description, URDF)
Before this commit: robot mycobot_description/urdf/ultraArm_p1, 15 links, 14 joints
Links:
- removed link J1-LINK
- removed link J2-Link3
- removed link J3-LIink2
- added link J1_LINK, mass 0.36023578514819; collision mesh filename=package://mycobot_description/urdf/ultraArm_p1/J1_LINK.STL; visual mesh filename=package://mycobot_description/urdf/ultraArm_p1/J1_LINK.STL
- added link J2_Link3, mass 0.000785398163397449; collision mesh filename=package://mycobot_description/urdf/ultraArm_p1/J2_Link3.STL; visual mesh filename=package://mycobot_description/urdf/ultraArm_p1/J2_Link3.STL
- added link J3_LIink2, mass 0.0559892080648003; collision mesh filename=package://mycobot_description/urdf/ultraArm_p1/J3_LIink2.STL; visual mesh filename=package://mycobot_description/urdf/ultraArm_p1/J3_LIink2.STL
Joints:
- removed joint J2-2
- removed joint J2-3
- removed joint J2-4
- removed joint J3-2
- removed joint J3-3
- removed joint J3-4
- added joint J2_2: type revolute, parent J1_LINK, child J2_Link2, origin xyz=-0.0025 -0.024 0.1049 rpy=0 0 0, axis 0 1 0, limit lower=-0.35 upper=1.3962 effort=100 velocity=1, mimic joint=J2 multiplier=1 offset=0
- added joint J2_3: type revolute, parent J2_Link2, child J2_Link3, origin xyz=0 0 0.14 rpy=0 0 0, axis 0 1 0, limit lower=1.3962 upper=0.35 effort=100 velocity=1, mimic joint=J2 multiplier=-1 offset=0
- added joint J2_4: type revolute, parent J2_Link1, child J2_Link4, origin xyz=-0.002409 0.0059 0.13998 rpy=0 0 0, axis 0 1 0, limit lower=-1.3962 upper=0.35 effort=100 velocity=1, mimic joint=J2_3 multiplier=1 offset=0
- added joint J3_2: type revolute, parent FIX3, child J3_LIink2, origin xyz=0 0 0 rpy=0 0 0, axis 0 1 0, limit lower=0 upper=1.92 effort=100 velocity=1, mimic joint=J3 multiplier=1 offset=0
- added joint J3_3: type revolute, parent J3_Link1, child J3_Link3, origin xyz=0.14232 -0.0099 -0.0049908 rpy=0 0 0, axis 0 1 0, limit lower=-1.92 upper=0 effort=100 velocity=1, mimic joint=J3 multiplier=-1 offset=0
- added joint J3_4: type revolute, parent J3_LIink2, child J3_Link4, origin xyz=0.13991 0.005 -0.0050135 rpy=0 0 0, axis 0 1 0, limit lower=-1.92 upper=0 effort=100 velocity=1, mimic joint=J3_3 multiplier=1 offset=0
- joint J1: child J1-LINK -> J1_LINK
- joint J2: parent J1-LINK -> J1_LINK

Commit message: perf(p1-ros2):Update URDF joint limits and update function package code.

File: mycobot_description/urdf/ultraArm_p1/ultraArm_p1.urdf (robot description, URDF)
Before this commit: robot firefighter, 15 links, 14 joints
Joints:
- joint J1: limit lower=-2.97 upper=2.97 effort=100 velocity=1 -> lower=-2.87 upper=2.87 effort=100 velocity=1
- joint J2: limit lower=-0.35 upper=1.3962 effort=100 velocity=1 -> lower=-0.31 upper=1.48 effort=100 velocity=1
- joint J2_2: limit lower=-0.35 upper=1.3962 effort=100 velocity=1 -> lower=-0.31 upper=1.48 effort=100 velocity=1
- joint J2_3: limit lower=1.3962 upper=0.35 effort=100 velocity=1 -> lower=1.48 upper=0.31 effort=100 velocity=1
- joint J2_4: limit lower=-1.3962 upper=0.35 effort=100 velocity=1 -> lower=-1.48 upper=0.31 effort=100 velocity=1
- joint J3: limit lower=0 upper=1.92 effort=100 velocity=1 -> lower=0 upper=1.49 effort=100 velocity=1
- joint J3_2: limit lower=0 upper=1.92 effort=100 velocity=1 -> lower=0 upper=1.49 effort=100 velocity=1
- joint J3_3: limit lower=-1.92 upper=0 effort=100 velocity=1 -> lower=-1.49 upper=0 effort=100 velocity=1
- joint J3_4: limit lower=-1.92 upper=0 effort=100 velocity=1 -> lower=-1.49 upper=0 effort=100 velocity=1
- joint J4: limit lower=-3.14 upper=3.14 effort=100 velocity=1 -> lower=-3.12 upper=3.12 effort=100 velocity=1

Commit message: fix(p1-ros2):Fixed some test bugs.

File: mycobot_description/urdf/ultraArm_p1/ultraArm_p1.urdf (robot description, URDF)
Before this commit: robot firefighter, 15 links, 14 joints
Joints:
- joint J3: limit lower=0 upper=1.49 effort=100 velocity=1 -> lower=0 upper=1.91 effort=100 velocity=1
- joint J3_2: limit lower=0 upper=1.49 effort=100 velocity=1 -> lower=0 upper=1.91 effort=100 velocity=1
- joint J3_3: limit lower=-1.49 upper=0 effort=100 velocity=1 -> lower=-1.91 upper=0 effort=100 velocity=1
- joint J3_4: limit lower=-1.49 upper=0 effort=100 velocity=1 -> lower=-1.91 upper=0 effort=100 velocity=1
