Commit message: feat(p1-ros2):Update the structure to the new version of the URDF model file

File: mycobot_description/urdf/ultraArm_p1/ultraArm_p1.urdf (robot description, URDF)
Before this commit: robot firefighter, 15 links, 14 joints
Links:
- removed link FIX1
- removed link FIX2
- removed link FIX3
- removed link J1_LINK
- removed link J2_Link1
- removed link J2_Link2
- removed link J2_Link3
- removed link J2_Link4
- removed link J3_LIink2
- removed link J3_Link1
- removed link J3_Link3
- removed link J3_Link4
- added link CENTER_V_2_Link, mass 0.0558803270642906; collision mesh filename=package://mycobot_description/urdf/ultraArm_p1/CENTER_V_2_L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; visual mesh filename=package://mycobot_description/urdf/ultraArm_p1/CENTER_V_2_L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
- added link FIX2_Link, mass 0.000117809724509617; collision mesh filename=package://mycobot_description/urdf/ultraArm_p1/FIX2_Link.STL; visual mesh filename=package://mycobot_description/urdf/ultraArm_p1/FIX2_Link.STL
- added link J1_Link, mass 0.390185141585949; collision mesh filename=package://mycobot_description/urdf/ultraArm_p1/J1_Link.STL; visual mesh filename=package://mycobot_description/urdf/ultraArm_p1/J1_Link.STL
- added link J2_2_Link, mass 0.0673595203554836; collision mesh filename=package://mycobot_description/urdf/ultraArm_p1/J2_2_Link.STL; visual mesh filename=package://mycobot_description/urdf/ultraArm_p1/J2_2_Link.STL
- added link J2_Link, mass 0.0395822221402214; collision mesh filename=package://mycobot_description/urdf/ultraArm_p1/J2_Link.STL; visual mesh filename=package://mycobot_description/urdf/ultraArm_p1/J2_Link.STL
- added link J3_4_Link, mass 0.000117809724509617; collision mesh filename=package://mycobot_description/urdf/ultraArm_p1/J3_4_Link.STL; visual mesh filename=package://mycobot_description/urdf/ultraArm_p1/J3_4_Link.STL
- added link J3_5_Link, mass 0.0663947658214263; collision mesh filename=package://mycobot_description/urdf/ultraArm_p1/J3_5_Link.STL; visual mesh filename=package://mycobot_description/urdf/ultraArm_p1/J3_5_Link.STL
- added link J3_Link, mass 0.0238706707614233; collision mesh filename=package://mycobot_description/urdf/ultraArm_p1/J3_Link.STL; visual mesh filename=package://mycobot_description/urdf/ultraArm_p1/J3_Link.STL
- added link center_Link, mass 0.0349898434561973; collision mesh filename=package://mycobot_description/urdf/ultraArm_p1/center_Link.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; visual mesh filename=package://mycobot_description/urdf/ultraArm_p1/center_Link.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
- added link center_v_1_Link, mass 0.000117809724509617; collision mesh filename=package://mycobot_description/urdf/ultraArm_p1/center_v_1_L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; visual mesh filename=package://mycobot_description/urdf/ultraArm_p1/center_v_1_L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
- added link fix1_Link, mass 0.000117809724509617; collision mesh filename=package://mycobot_description/urdf/ultraArm_p1/fix1_Link.STL; visual mesh filename=package://mycobot_description/urdf/ultraArm_p1/fix1_Link.STL
- link J4_Link: mass 0.00784859322698103 -> 0.00948835945053853
- link base_link: mass 0.627583870747359 -> 0.435296505947694
Joints:
- removed joint F1
- removed joint F2
- removed joint F3
- removed joint J2_3
- removed joint J2_4
- removed joint J3_2
- removed joint J3_3
- added joint CENTER_V_2: type revolute, parent center_Link, child CENTER_V_2_Link, origin xyz=0.00015 0.025 0.025 rpy=0 0 0, axis -1 0 0, limit lower=-0.017 upper=1.91 effort=0 velocity=0, mimic joint=J3 multiplier=1 offset=0
- added joint FIX2: type fixed, parent J3_5_Link, child FIX2_Link, origin xyz=0.0104999999999947 0.025000000023119 0.0249999447386166 rpy=0 0 0, axis 0 0 0
- added joint J3_5: type revolute, parent J3_Link, child J3_5_Link, origin xyz=0.0055 0.14 0 rpy=0 0 0, axis -1 0 0, limit lower=-1.91 upper=0.017 effort=0 velocity=0, mimic joint=J3 multiplier=-1 offset=0
- added joint center: type revolute, parent J2_Link, child center_Link, origin xyz=0.00335 -0.00036008 0.14036 rpy=0 0 0, axis -1 0 0, limit lower=-1.48 upper=0.31 effort=0 velocity=0, mimic joint=J2 multiplier=-1 offset=0
- added joint center_v_1: type revolute, parent J2_2_Link, child center_v_1_Link, origin xyz=-0.0045 0 0.14 rpy=0 0 0, axis -1 0 0, limit lower=-1.48 upper=0.31 effort=0 velocity=0, mimic joint=J2 multiplier=-1 offset=0
- added joint fix1: type fixed, parent center_Link, child fix1_Link, origin xyz=0.000149999999997076 -0.0250000000000165 0.0249999999999976 rpy=0 0 0, axis 0 0 0
- joint J1: child J1_LINK -> J1_Link; limit lower=-2.87 upper=2.87 effort=100 velocity=1 -> lower=-2.87 upper=2.87 effort=0 velocity=0; origin xyz=0 0 0.0860000000000012 rpy=0 0 0 -> xyz=-0.000100404778856366 0 0.0859999999999997 rpy=0 0 0
- joint J2: axis 0 1 0 -> -1 0 0; child J2_Link1 -> J2_Link; limit lower=-0.31 upper=1.48 effort=100 velocity=1 -> lower=-0.31 upper=1.48 effort=0 velocity=0; origin xyz=0.0225 -0.015 0.0799 rpy=0 0 0 -> xyz=0.0161 0.02286 0.079544 rpy=0 0 0; parent J1_LINK -> J1_Link
- joint J2_2: axis 0 1 0 -> -1 0 0; child J2_Link2 -> J2_2_Link; limit lower=-0.31 upper=1.48 effort=100 velocity=1 -> lower=-0.31 upper=1.48 effort=0 velocity=0; origin xyz=-0.0025 -0.024 0.1049 rpy=0 0 0 -> xyz=0.0241 -0.0025 0.1049 rpy=0 0 0; parent J1_LINK -> J1_Link
- joint J3: axis 0 1 0 -> -1 0 0; child J3_Link1 -> J3_Link; limit lower=0 upper=1.91 effort=100 velocity=1 -> lower=-0.017 upper=1.91 effort=0 velocity=0; origin xyz=0 0 0 rpy=0 0 0 -> xyz=-0.01485 0 0 rpy=0 0 0; parent J2_Link4 -> center_Link
- joint J3_4: axis 0 1 0 -> -1 0 0; child J3_Link4 -> J3_4_Link; limit lower=-1.91 upper=0 effort=100 velocity=1 -> lower=-1.91 upper=0.017 effort=0 velocity=0; mimic joint=J3_3 multiplier=1 offset=0 -> joint=J3 multiplier=-1 offset=0; origin xyz=0.13991 0.005 -0.0050135 rpy=0 0 0 -> xyz=0.001 0.14 0 rpy=0 0 0; parent J3_LIink2 -> CENTER_V_2_Link
- joint J4: axis 3.005E-05 0 1 -> 0 0 -1; limit lower=-3.12 upper=3.12 effort=100 velocity=1 -> lower=-3.12 upper=3.12 effort=0 velocity=0; origin xyz=0.067813 0.019 -0.047739 rpy=0 0 0 -> xyz=-0.00950000000000579 0.0609999386572151 -0.0305000950662462 rpy=0 0 0; parent J3_Link3 -> J3_5_Link

Commit message: Repair J4 motion direction

File: mycobot_description/urdf/ultraArm_p1/ultraArm_p1.urdf (robot description, URDF)
Before this commit: robot firefighter, 14 links, 13 joints
Joints:
- joint J4: axis 0 0 -1 -> 0 0 1
