Commit message: fix: joint angle limits in URDF

File: mycobot_description/urdf/mycobot_pro_600/mycobot_pro_600.urdf (robot description, URDF)
Before this commit: robot firefighter, 7 links, 6 joints
Joints:
- joint joint3_to_joint2: limit lower=-3.14159 upper=3.14159 effort=1000.0 velocity=0 -> lower=-4.7123 upper=1.5708 effort=1000.0 velocity=0
- joint joint4_to_joint3: limit lower=-2.6179 upper=2.443 effort=1000.0 velocity=0 -> lower=-2.6179 upper=2.6179 effort=1000.0 velocity=0
- joint joint5_to_joint4: limit lower=-2.9670 upper=2.9670 effort=1000.0 velocity=0 -> lower=-4.5378 upper=1.3962 effort=1000.0 velocity=0
