Commit message: fix: fix collision volume, add speed settings, and optimize UI

File: mycobot_pro/mycobotpro450_gazeboros2/config/mycobot_pro_450_force_gripper.urdf (robot description, URDF)
Before this commit: robot firefighter, 16 links, 15 joints
Links:
- link base: geometry collision mesh filename=package://mycobot_description/urdf/mycobot_pro_450/collisio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; visual mesh filename=package://mycobot_description/urdf/mycobot_pro_450/PRO450_J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
- link gripper_base: geometry collision mesh filename=package://mycobot_description/urdf/mycobot_pro_450/collisio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; visual mesh filename=package://mycobot_description/urdf/mycobot_320_m5_2022/forc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
- link gripper_connection: geometry collision mesh filename=package://mycobot_description/urdf/mycobot_pro_450/collisio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; visual mesh filename=package://mycobot_description/urdf/mycobot_320_m5_2022/forc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
- link gripper_left1: geometry collision mesh filename=package://mycobot_description/urdf/mycobot_pro_450/collisio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; visual mesh filename=package://mycobot_description/urdf/mycobot_320_m5_2022/forc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
- link gripper_left2: geometry collision mesh filename=package://mycobot_description/urdf/mycobot_pro_450/collisio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; visual mesh filename=package://mycobot_description/urdf/mycobot_320_m5_2022/forc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
- link gripper_left3: geometry collision mesh filename=package://mycobot_description/urdf/mycobot_pro_450/collisio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; visual mesh filename=package://mycobot_description/urdf/mycobot_320_m5_2022/forc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
- link gripper_right1: geometry collision mesh filename=package://mycobot_description/urdf/mycobot_pro_450/collisio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; visual mesh filename=package://mycobot_description/urdf/mycobot_320_m5_2022/forc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
- link gripper_right2: geometry collision mesh filename=package://mycobot_description/urdf/mycobot_pro_450/collisio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; visual mesh filename=package://mycobot_description/urdf/mycobot_320_m5_2022/forc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
- link gripper_right3: geometry collision mesh filename=package://mycobot_description/urdf/mycobot_pro_450/collisio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; visual mesh filename=package://mycobot_description/urdf/mycobot_320_m5_2022/forc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
- link link1: geometry collision mesh filename=package://mycobot_description/urdf/mycobot_pro_450/collisio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; visual mesh filename=package://mycobot_description/urdf/mycobot_pro_450/PRO450_J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
- link link2: geometry collision mesh filename=package://mycobot_description/urdf/mycobot_pro_450/collisio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; visual mesh filename=package://mycobot_description/urdf/mycobot_pro_450/PRO450_J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
- link link3: geometry collision mesh filename=package://mycobot_description/urdf/mycobot_pro_450/collisio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; visual mesh filename=package://mycobot_description/urdf/mycobot_pro_450/PRO450_J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
- link link4: geometry collision mesh filename=package://mycobot_description/urdf/mycobot_pro_450/collisio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; visual mesh filename=package://mycobot_description/urdf/mycobot_pro_450/PRO450_J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
- link link5: geometry collision mesh filename=package://mycobot_description/urdf/mycobot_pro_450/collisio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; visual mesh filename=package://mycobot_description/urdf/mycobot_pro_450/PRO450_J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
- link link6: geometry collision mesh filename=package://mycobot_description/urdf/mycobot_pro_450/collisio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; visual mesh filename=package://mycobot_description/urdf/mycobot_pro_450/PRO450_J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

Commit message: perf: optimize collision matrix for random motion

File: mycobot_pro/mycobotpro450_gazeboros2/config/mycobot_pro_450_force_gripper.urdf (robot description, URDF)
Before this commit: robot firefighter, 16 links, 15 joints
Links:
- added link gripper_cable_terminal, mass 0.000001; collision cylinder length=0.020 radius=0.006624266
Joints:
- added joint gripper_base_to_cable_terminal: type fixed, parent gripper_base, child gripper_cable_terminal, origin xyz=-0.107 0.012 0.0 rpy=1.5708 0 1.5708

Commit message: perf: optimize functionality and execution logic

File: mycobot_pro/mycobotpro450_gazeboros2/config/mycobot_pro_450_force_gripper.urdf (robot description, URDF)
Before this commit: robot firefighter, 17 links, 16 joints
Links:
- link gripper_cable_terminal: geometry collision cylinder length=0.025 radius=0.006624266
