Commit message: Add files via upload

File: mycobot_pro/mycobotpro450_gazeboros2/config/firefighter.ros2_control.xacro (robot description, xacro)
@@ -57,34 +57,4 @@
                 <state_interface name="velocity"/>
             </joint>
-            <joint name="gripper_base_to_gripper_left2">
-                <param name="mimic">gripper_controller</param>
-                <param name="multiplier">1.0</param>
-                <command_interface name="position"/>
-                <state_interface name="position"/>
-            </joint>
-            <joint name="gripper_left3_to_gripper_left1">
-                <param name="mimic">gripper_controller</param>
-                <param name="multiplier">-1.0</param>
-                <command_interface name="position"/>
-                <state_interface name="position"/>
-            </joint>
-            <joint name="gripper_base_to_gripper_right3">
-                <param name="mimic">gripper_controller</param>
-                <param name="multiplier">-1.0</param>
-                <command_interface name="position"/>
-                <state_interface name="position"/>
-            </joint>
-            <joint name="gripper_base_to_gripper_right2">
-                <param name="mimic">gripper_controller</param>
-                <param name="multiplier">-1.0</param>
-                <command_interface name="position"/>
-                <state_interface name="position"/>
-            </joint>
-            <joint name="gripper_right3_to_gripper_right1">
-                <param name="mimic">gripper_controller</param>
-                <param name="multiplier">1.0</param>
-                <command_interface name="position"/>
-                <state_interface name="position"/>
-            </joint>
         </ros2_control>
     </xacro:macro>

File: mycobot_pro/mycobotpro450_gazeboros2/config/mycobot_pro_450_force_gripper.urdf (robot description, URDF)
Before this commit: robot firefighter, 16 links, 15 joints
Links:
- link base: mass 1000.0 -> 8.0
- link gripper_base: mass 0.005 -> 0.12
- link gripper_connection: mass 0.1 -> 0.15
- link gripper_left1: mass 0.005 -> 0.02
- link gripper_left2: mass 0.005 -> 0.02
- link gripper_left3: mass 0.005 -> 0.02
- link gripper_right1: mass 0.005 -> 0.02
- link gripper_right2: mass 0.005 -> 0.02
- link gripper_right3: mass 0.005 -> 0.02
- link link1: mass 20.0 -> 3.5
- link link2: mass 1.0 -> 2.8
- link link3: mass 2.0 -> 2.2
- link link4: mass 1.0 -> 1.2
- link link5: mass 1.0 -> 0.8
- link link6: mass 1.0 -> 0.4
Joints:
- joint joint3: origin xyz=-0.01 0 0.18   rpy=0 0 0 -> xyz=-0.01 0 0.18 rpy=0 0 0

Commit message: perf: optimize gripper collision matrix for random motion and UI

File: mycobot_pro/mycobotpro450_gazeboros2/config/firefighter.ros2_control.xacro (robot description, xacro)
@@ -57,4 +57,52 @@
                 <state_interface name="velocity"/>
             </joint>
+            <!-- Keep all gripper joints in the same GazeboSystem update.
+                 The separate mimic plugins set fmax to the effort limit and
+                 changed positions without resetting their residual velocity. -->
+            <joint name="gripper_base_to_gripper_left2">
+                <param name="mimic">gripper_controller</param>
+                <param name="multiplier">1.0</param>
+                <command_interface name="position"/>
+                <state_interface name="position">
+                  <param name="initial_value">${initial_positions['gripper_controller']}</param>
+                </state_interface>
+                <state_interface name="velocity"/>
+            </joint>
+            <joint name="gripper_left3_to_gripper_left1">
+                <param name="mimic">gripper_controller</param>
+                <param name="multiplier">-1.0</param>
+                <command_interface name="position"/>
+                <state_interface name="position">
+                  <param name="initial_value">${-initial_positions['gripper_controller']}</param>
+                </state_interface>
+                <state_interface name="velocity"/>
+            </joint>
+            <joint name="gripper_base_to_gripper_right3">
+                <param name="mimic">gripper_controller</param>
+                <param name="multiplier">-1.0</param>
+                <command_interface name="position"/>
+                <state_interface name="position">
+                  <param name="initial_value">${-initial_positions['gripper_controller']}</param>
+                </state_interface>
+                <state_interface name="velocity"/>
+            </joint>
+            <joint name="gripper_base_to_gripper_right2">
+                <param name="mimic">gripper_controller</param>
+                <param name="multiplier">-1.0</param>
+                <command_interface name="position"/>
+                <state_interface name="position">
+                  <param name="initial_value">${-initial_positions['gripper_controller']}</param>
+                </state_interface>
+                <state_interface name="velocity"/>
+            </joint>
+            <joint name="gripper_right3_to_gripper_right1">
+                <param name="mimic">gripper_controller</param>
+                <param name="multiplier">1.0</param>
+                <command_interface name="position"/>
+                <state_interface name="position">
+                  <param name="initial_value">${initial_positions['gripper_controller']}</param>
+                </state_interface>
+                <state_interface name="velocity"/>
+            </joint>
         </ros2_control>
     </xacro:macro>

File: mycobot_pro/mycobotpro450_gazeboros2/config/mycobot_pro_450_force_gripper.urdf (robot description, URDF)
Before this commit: robot firefighter, 17 links, 16 joints
Joints:
- joint joint6: origin xyz=0 0.04 0.0435 rpy=0.7853981634 0 1.5708 -> xyz=0 0.04 0.0435 rpy=2.3561944901948966 0 1.5708
- joint joint6_to_gripper_connect: origin xyz=0.03 0.0 -0.01 rpy=-1.5708 0 -1.5708 -> xyz=0.03 -0.01 0 rpy=-0.0000036732217733577977 -1.5707926535897934 -3.1415926535731233

Commit message: feat: add support for grippers with and without force control

File: mycobot_pro/mycobotpro450_gazeboros2/config/firefighter.ros2_control.xacro (robot description, xacro)
@@ -50,4 +50,5 @@
                 <state_interface name="velocity"/>
             </joint>
+            <xacro:if value="$(arg with_gripper)">
             <joint name="gripper_controller">
                 <command_interface name="position"/>
@@ -105,4 +106,5 @@
                 <state_interface name="velocity"/>
             </joint>
+            </xacro:if>
         </ros2_control>
     </xacro:macro>

File: mycobot_pro/mycobotpro450_gazeboros2/config/firefighter.urdf.xacro (robot description, xacro)
@@ -1,4 +1,6 @@
 <?xml version="1.0"?>
 <robot xmlns:xacro="http://www.ros.org/wiki/xacro" name="firefighter">
+    <xacro:arg name="with_gripper" default="true" />
+    <xacro:arg name="controller_config_file" default="$(find mycobotpro450_gazeboros2)/config/ros2_controllers.yaml" />
     <xacro:arg name="initial_positions_file" default="initial_positions.yaml" />
     <!-- MoveIt uses collision_exact by default. Gazebo overrides this with
@@ -13,5 +15,5 @@
     <gazebo>
         <plugin filename="libgazebo_ros2_control.so" name="gazebo_ros2_control">
-            <parameters>$(find mycobotpro450_gazeboros2)/config/ros2_controllers.yaml</parameters>
+            <parameters>$(arg controller_config_file)</parameters>
             <!-- The Gazebo entity is spawned from the namespaced description
                  publisher because it uses collision_gazebo and, in real-pose

File: mycobot_pro/mycobotpro450_gazeboros2/config/mycobot_pro_450_force_gripper.urdf (robot description, URDF)
Before this commit: robot firefighter, 17 links, 16 joints
Links:
- removed link gripper_base
- removed link gripper_cable_terminal
- removed link gripper_connection
- removed link gripper_left1
- removed link gripper_left2
- removed link gripper_left3
- removed link gripper_right1
- removed link gripper_right2
- removed link gripper_right3
Joints:
- removed joint gripper_base_to_cable_terminal
- removed joint gripper_base_to_gripper_left2
- removed joint gripper_base_to_gripper_right2
- removed joint gripper_base_to_gripper_right3
- removed joint gripper_controller
- removed joint gripper_left3_to_gripper_left1
- removed joint gripper_right3_to_gripper_right1
- removed joint joint6_to_gripper_base
- removed joint joint6_to_gripper_connect
