Commit message: refactor: optimize collision volume detection

File: mycobot_pro/mycobotpro450_gazeboros2/config/firefighter.urdf.xacro (robot description, xacro)
@@ -2,4 +2,8 @@
 <robot xmlns:xacro="http://www.ros.org/wiki/xacro" name="firefighter">
     <xacro:arg name="initial_positions_file" default="initial_positions.yaml" />
+    <!-- MoveIt uses collision_exact by default. Gazebo overrides this with
+         collision_gazebo because ODE is unstable with dynamic non-convex,
+         high-triangle collision meshes. -->
+    <xacro:arg name="collision_mesh_dir" default="collision_exact" />
     <!-- Import firefighter urdf file -->
     <xacro:include filename="$(find mycobotpro450_gazeboros2)/config/mycobot_pro_450_force_gripper.urdf" />

File: mycobot_pro/mycobotpro450_gazeboros2/config/mycobot_pro_450_force_gripper.urdf (robot description, URDF)
Before this commit: robot firefighter, 16 links, 15 joints
Links:
- link base: geometry collision mesh filename=package://mycobot_description/urdf/mycobot_pro_450/$(arg co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; visual mesh filename=package://mycobot_description/urdf/mycobot_pro_450/PRO450_J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
- link gripper_base: geometry collision mesh filename=package://mycobot_description/urdf/mycobot_pro_450/$(arg co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; visual mesh filename=package://mycobot_description/urdf/mycobot_320_m5_2022/forc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
- link gripper_connection: geometry collision mesh filename=package://mycobot_description/urdf/mycobot_pro_450/$(arg co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; visual mesh filename=package://mycobot_description/urdf/mycobot_320_m5_2022/forc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
- link gripper_left1: geometry collision mesh filename=package://mycobot_description/urdf/mycobot_pro_450/$(arg co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; visual mesh filename=package://mycobot_description/urdf/mycobot_320_m5_2022/forc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
- link gripper_left2: geometry collision mesh filename=package://mycobot_description/urdf/mycobot_pro_450/$(arg co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; visual mesh filename=package://mycobot_description/urdf/mycobot_320_m5_2022/forc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
- link gripper_left3: geometry collision mesh filename=package://mycobot_description/urdf/mycobot_pro_450/$(arg co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; visual mesh filename=package://mycobot_description/urdf/mycobot_320_m5_2022/forc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
- link gripper_right1: geometry collision mesh filename=package://mycobot_description/urdf/mycobot_pro_450/$(arg co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; visual mesh filename=package://mycobot_description/urdf/mycobot_320_m5_2022/forc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
- link gripper_right2: geometry collision mesh filename=package://mycobot_description/urdf/mycobot_pro_450/$(arg co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; visual mesh filename=package://mycobot_description/urdf/mycobot_320_m5_2022/forc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
- link gripper_right3: geometry collision mesh filename=package://mycobot_description/urdf/mycobot_pro_450/$(arg co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; visual mesh filename=package://mycobot_description/urdf/mycobot_320_m5_2022/forc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
- link link1: geometry collision mesh filename=package://mycobot_description/urdf/mycobot_pro_450/$(arg co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; visual mesh filename=package://mycobot_description/urdf/mycobot_pro_450/PRO450_J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
- link link2: geometry collision mesh filename=package://mycobot_description/urdf/mycobot_pro_450/$(arg co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; visual mesh filename=package://mycobot_description/urdf/mycobot_pro_450/PRO450_J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
- link link3: geometry collision mesh filename=package://mycobot_description/urdf/mycobot_pro_450/$(arg co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; visual mesh filename=package://mycobot_description/urdf/mycobot_pro_450/PRO450_J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
- link link4: geometry collision mesh filename=package://mycobot_description/urdf/mycobot_pro_450/$(arg co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; visual mesh filename=package://mycobot_description/urdf/mycobot_pro_450/PRO450_J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
- link link5: geometry collision mesh filename=package://mycobot_description/urdf/mycobot_pro_450/$(arg co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; visual mesh filename=package://mycobot_description/urdf/mycobot_pro_450/PRO450_J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
- link link6: geometry collision mesh filename=package://mycobot_description/urdf/mycobot_pro_450/$(arg co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; visual mesh filename=package://mycobot_description/urdf/mycobot_pro_450/PRO450_J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

Commit message: feat: add keyboard control and real robot link

File: mycobot_pro/mycobotpro450_gazeboros2/config/firefighter.urdf.xacro (robot description, xacro)
@@ -14,4 +14,11 @@
         <plugin filename="libgazebo_ros2_control.so" name="gazebo_ros2_control">
             <parameters>$(find mycobotpro450_gazeboros2)/config/ros2_controllers.yaml</parameters>
+            <!-- The Gazebo entity is spawned from the namespaced description
+                 publisher because it uses collision_gazebo and, in real-pose
+                 mirror mode, the read-only hardware snapshot.  Do not let the
+                 plugin fall back to the MoveIt robot_state_publisher, whose
+                 ros2_control initial values are the default zero pose. -->
+            <robot_param>robot_description</robot_param>
+            <robot_param_node>/gazebo_spawn/robot_description_publisher</robot_param_node>
         </plugin>
     </gazebo>

File: mycobot_pro/mycobotpro450_gazeboros2/config/mycobot_pro_450_force_gripper.urdf (robot description, URDF)
Before this commit: robot firefighter, 16 links, 15 joints
Joints:
- joint joint6: origin xyz=0 0.04 0.0435 rpy=0 0 1.5708 -> xyz=0 0.04 0.0435 rpy=0.7853981634 0 1.5708

Commit message: fix: resolve model bugs

File: mycobot_pro/mycobotpro450_gazeboros2/config/firefighter.urdf.xacro (robot description, xacro)
@@ -2,4 +2,6 @@
 <robot xmlns:xacro="http://www.ros.org/wiki/xacro" name="firefighter">
     <xacro:arg name="with_gripper" default="true" />
+    <!-- Internal mirror setting; simulation and MoveIt retain normal collisions. -->
+    <xacro:arg name="gazebo_contact_response" default="true" />
     <xacro:arg name="controller_config_file" default="$(find mycobotpro450_gazeboros2)/config/ros2_controllers.yaml" />
     <xacro:arg name="initial_positions_file" default="initial_positions.yaml" />

File: mycobot_pro/mycobotpro450_gazeboros2/config/mycobot_pro_450_force_gripper.urdf (robot description, URDF)
Before this commit: robot firefighter, 8 links, 7 joints
Joints:
- joint joint1: origin xyz=-0.0045 0 0.155 rpy=0 0 0 -> xyz=-0.003696284968 -0.000524188133 0.162208908081 rpy=0 0 0
- joint joint2: origin xyz=0.05 0 0.048 rpy=0 0 0 -> xyz=0.047000183626 -0.000000172583 0.049999827418 rpy=0 0 0
- joint joint3: origin xyz=-0.01 0 0.18 rpy=0 0 0 -> xyz=-0.004000003825 0.000002823248 0.179999372705 rpy=0 0 0
- joint joint4: origin xyz=0.0 0 0.1735 rpy=0 0 0 -> xyz=-0.005999977121 0.000002620318 0.172999270259 rpy=0 0 0
- joint joint5: origin xyz=0.046 0.0003 0.05 rpy=0 0 0 -> xyz=0.047989648139 0.000003599231 0.054000176186 rpy=0 0 0
- joint joint6: origin xyz=0 0.04 0.0435 rpy=2.3561944901948966 0 1.5708 -> xyz=-0.000002439502 0.039949245866 0.042500131832 rpy=2.3561944901948966 0 1.5708
