Commit message: refactor: modify GUI input threshold

File: mycobot_pro/mycobotpro630_gazeboros2/config/mycobot_pro_630_force_gripper.urdf (robot description, URDF)
Before this commit: robot firefighter, 8 links, 7 joints
Joints:
- joint joint1_to_base: limit lower=-3.14 upper=3.14159 effort=1000.0 velocity=3.14 -> lower=-3.141592653589793 upper=3.141592653589793 effort=1000.0 velocity=3.14
- joint joint2_to_joint1: limit lower=-3.14159 upper=3.14159 effort=1000.0 velocity=3.14 -> lower=-3.141592653589793 upper=3.141592653589793 effort=1000.0 velocity=3.14
- joint joint3_to_joint2: limit lower=-2.61 upper=2.618 effort=1000.0 velocity=3.14 -> lower=-2.6179938779914944 upper=2.6179938779914944 effort=1000.0 velocity=3.14
- joint joint4_to_joint3: limit lower=-2.9670 upper=2.9670 effort=1000.0 velocity=3.14 -> lower=-2.9670597283903604 upper=2.9670597283903604 effort=1000.0 velocity=3.14
- joint joint5_to_joint4: limit lower=-2.93 upper=2.9321 effort=1000.0 velocity=3.14 -> lower=-2.9321531433504737 upper=2.9321531433504737 effort=1000.0 velocity=3.14
- joint joint6_to_joint5: limit lower=-3.03 upper=3.0368 effort=1000.0 velocity=3.14 -> lower=-3.036872898470133 upper=3.036872898470133 effort=1000.0 velocity=3.14
